File: Electronics/OpenThereminV45.kicad_sch (KiCad schematic)
At the start: 99 parts, among them J1 USB_C_Receptacle 12401610E4#2A, J2 Conn_02x03_Odd_Even, J3 Conn_02x05_Odd_Even, P1 10k, P10 BUTTON, P11 A3_PAD, P12 A2_PAD, P13 A1_PAD, P14 A0_PAD, P16 GND, P2 10k, P3 10k, P4 10k, P8 VCC, P9 GND, U1 TTP223, U10 CH340C, U11 LP2985-3.3, U12 MCP4922-E/SL, U2 74HC4060D, U3 74HC4060D, U4 74HC74, U5 HEF4069, U6 MCP4921-E/SN, U7 MCP4922-E/SL, U8 MCP6002T-I/SN, U9 ATmega328P-AU, X1 16MHz, X2 7.3721MHz, Y1 MountPad3, Y2 MountPad3, Y3 PLUG_3_5_SMD SJ-3502-SMT-TR, Y7 PLUG_3_5_SMD SJ-3502-SMT-TR

Commit message: changed to 4-layer and added esd protection and bypass caps
not final yet, audio connector has wrong footprint
Parts:
- added C19, C31, C39: 100nF, Capacitor_SMD:C_0603_1608Metric, symbol OpenThereminV41-rescue:C-OpenThereminV4-rescue
- added C40: 100n, Capacitor_SMD:C_0603_1608Metric, symbol OpenThereminV41-rescue:C-OpenThereminV4-rescue
- added C41: 10u, Capacitor_SMD:C_0603_1608Metric, symbol OpenThereminV41-rescue:C-OpenThereminV4-rescue
- added D4: PRTR5V0U2X, Package_TO_SOT_SMD:SOT-143, symbol Power_Protection:PRTR5V0U2X
- added D5, D6, D7, D8: PESD5V0X1BL, Diode_SMD:D_SOD-882, symbol Device:D_TVS
- added R23, R24: 10R, Resistor_SMD:R_0603_1608Metric, symbol OpenThereminV41-rescue:RES-OpenThereminV4-rescue
- C4, U12: now not fitted
- D3: value DualLED 156125RB73000 -> DualLED 156125RB73000
- GROUND1, W1, W2, Y1, Y2: now left out of the parts list
- J1: value USB_C_Receptacle 12401610E4#2A -> USB_C_Receptacle 12401610E4#2A
- U4: value 74HC74 -> 74HC74D
- Y3: value PLUG_3_5_SMD SJ-3502-SMT-TR -> PLUG_3_5_SMD SJ-3502-SMT-TR; now not fitted
- Y7: value PLUG_3_5_SMD SJ-3502-SMT-TR -> PLUG_3_5_SMD SJ-3502-SMT-TR
Connections:
- net AUDIO: now also C29.1, R23.1, R24.1; no longer C29.2, Y7.3 (L)
- net D+: now also D4.2 (I/O1); no longer J3.9 (Pin_9)
- net D-: now also D4.3 (I/O2); no longer J3.8 (Pin_8)
- net GATE: now also D5.2 (A2)
- net GND: now also J1.S1 (SHIELD), C19.2, C31.2, C39.2, C40.2, C41.2, D4.1 (GND), D5.1 (A1), D6.2 (A2), D7.2 (A2), D8.1 (A1)
- net VCC: now also C19.1, C31.1, C39.1, C40.1, C41.1, D4.4 (VCC)
- net at C2.1, C4.1, C5.1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: now also D6.1 (A1)
- net at C11.1, C12.1, C9.1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: now also D7.1 (A1)
- net at C34.1, P10.1 (P1), U1.3 (I): now also D8.2 (A2)
- new net: C29.2, Y7.3 (L)
- new net: R23.2, U8.1, U8.2 (-)
- new net: R24.2, U8.6 (-), U8.7
- no-connect marks 0 -> 45
Other:
- moved on the sheet: C20, C29, C33, GROUND1, P10, P16, R15, R18, R19, U8B, Y7

Commit message: Added some text; moved some reference descriptors; pcb layer identification
Parts:
- added XX1, XX2, XX3, XX4: XEJPL5207CR, symbol Theremin:potmeter_shaft
Connections:
- net AUDIO: now also C29.2, Y7.3 (L); no longer C29.1, R23.1, R24.1
- new net: C29.1, R23.1, R24.1
Other:
- moved on the sheet: C30, C34, D5, D8, P1, P2, R20

Commit message: 4-layer version; 3D updates and more
Parts:
- removed W1: FIDUCIAL1, GaudiLabsFootPrints:Fiducial_1mm_Dia_2.54mm_Outer_CopperBottom, symbol OpenThereminV41-rescue:TEST_1P-OpenThereminV4-rescue
- removed W2: FIDUCIAL2, GaudiLabsFootPrints:Fiducial_1mm_Dia_2.54mm_Outer_CopperBottom, symbol OpenThereminV41-rescue:TEST_1P-OpenThereminV4-rescue
- added C42, C43, C44, C45: 100n, Capacitor_SMD:C_0603_1608Metric, symbol OpenThereminV41-rescue:C-OpenThereminV4-rescue
- added FID1, FID2, FID3: Fiducial, Fiducial:Fiducial_1mm_Mask3mm, symbol Mechanical:Fiducial
- added H1, H2, H3, H4: MountingHole, MountingHole:MountingHole_3.2mm_M3, symbol Mechanical:MountingHole
- added R25, R26: 0R, Resistor_SMD:R_0603_1608Metric, symbol OpenThereminV41-rescue:RES-OpenThereminV4-rescue
- C36, C37, C41: value 10u -> 10uF
- J1: value USB_C_Receptacle 12401610E4#2A -> 12401610E4#2A
- J2, J3: now not fitted
- L1, L2: footprint GaudiLabsFootPrints:COIL_T -> theremin-footprints:COIL_T
- P1, P2, P3, P4: value 10k -> PS15NV60-103A3030; footprint GaudiLabsFootPrints:PS15NV60 -> theremin-footprints:PS15NV60
- P10, P11, P12, P13, P14, P16, P8, P9: now left out of the parts list
- U1: value TTP223 -> TTP223E-BA6
- U11: value LP2985-3.3 -> LP2985-3.3DBV
- U5: value HEF4069 -> HEF4069UBT
- U9: value ATmega328P-AU -> ATMEGA328P-AU
- X1: value 16MHz -> 16MHz/30ppm/18pF
- X2: value 7.3721MHz -> 7.3721MHz/30ppm/18pF
- Y3, Y7: value PLUG_3_5_SMD SJ-3502-SMT-TR -> SJ-3523-SMT-TR
Connections:
- net A0: now also C42.1
- net A1: now also C43.1
- net A2: now also C44.1
- net A3: now also C45.1
- net AUDIO: now also R25.2
- net GATE: now also R26.2; no longer Y7.2 (R)
- net GND: now also C42.2, C43.2, C44.2, C45.2
- new net: R25.1, R26.1, Y7.2 (R)
- no-connect marks 45 -> 43
Other:
- note added: "If you want to use the CV1 and CV2 signals, place the DAC and the connector"
- note added: "place only one resistor: R25 for use of headphones (L+R) R26 for use of gate signal"
- note removed: "PS15NV60-103A3030"
- moved on the sheet: P1, P3, P4, XX1, XX2, XX3, XX4
